File: levelshifter/levelshifter.kicad_pcb (KiCad board)
At the start: 2 copper layers, 60 x 33 mm, 32 parts, among them J1 V_IN, J10 Terminal8, J11 Terminal9, J12 Terminal10, J2 V_OUT, J3 Terminal1, J4 Terminal2, J5 Terminal3, J6 Terminal4, J7 Terminal5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

Commit message: Many things
Parts:
- added J13: V_IN_1, Connector_PinHeader_2.54mm:PinHeader_1x02_P2.54mm_Vertical, F.Cu at (143.0, 68.0)
- added J14: V_IN_2, Connector_PinHeader_2.54mm:PinHeader_1x02_P2.54mm_Vertical, F.Cu at (149.0, 68.0)
- added J15: V_IN_3, Connector_PinHeader_2.54mm:PinHeader_1x02_P2.54mm_Vertical, F.Cu at (155.0, 68.0)
- added J16: V_IN_4, Connector_PinHeader_2.54mm:PinHeader_1x02_P2.54mm_Vertical, F.Cu at (161.0, 68.0)
- added J17: V_IN_5, Connector_PinHeader_2.54mm:PinHeader_1x02_P2.54mm_Vertical, F.Cu at (167.0, 68.0)
- added J18: V_IN_6, Connector_PinHeader_2.54mm:PinHeader_1x02_P2.54mm_Vertical, F.Cu at (173.0, 68.0)
- added J19: V_IN_7, Connector_PinHeader_2.54mm:PinHeader_1x02_P2.54mm_Vertical, F.Cu at (179.0, 68.0)
- added J20: V_IN_8, Connector_PinHeader_2.54mm:PinHeader_1x02_P2.54mm_Vertical, F.Cu at (185.0, 68.0)
- added J21: V_IN_9, Connector_PinHeader_2.54mm:PinHeader_1x02_P2.54mm_Vertical, F.Cu at (191.0, 68.0)
- added J22: V_IN_10, Connector_PinHeader_2.54mm:PinHeader_1x02_P2.54mm_Vertical, F.Cu at (197.0, 68.0)
Connections:
- net Net-(Q1-Pad1) renamed /In1
- net Net-(Q10-Pad1) renamed /In10
- net Net-(Q2-Pad1) renamed /In2
- net Net-(Q3-Pad1) renamed /In3
- net Net-(Q4-Pad1) renamed /In4
- net Net-(Q5-Pad1) renamed /In5
- net Net-(Q6-Pad1) renamed /In6
- net Net-(Q7-Pad1) renamed /In7
- net Net-(Q8-Pad1) renamed /In8
- net Net-(Q9-Pad1) renamed /In9
Routing:
- net /In9: track 3.53 -> 6.58 mm
- net /In8: track 3.53 -> 6.58 mm
- net /In7: track 3.53 -> 6.58 mm
- net /In6: track 3.53 -> 6.58 mm
- net /In5: track 3.53 -> 6.58 mm
- net /In4: track 3.53 -> 6.58 mm
- net /In3: track 3.53 -> 6.58 mm
- net /In2: track 3.53 -> 6.58 mm
- net /In10: track 3.53 -> 6.58 mm
